File: MACMOD.brd (EAGLE design)
At the start: 12.7 x 10.2 mm, 5 parts, among them IC1 MCP24AA025E48

Commit message: Improved labels for v1.0 release
Changed lines of the file:
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@@
 <text x="2.667" y="1.143" size="0.8128" layer="21" font="vector" ratio="17" rot="R90">5.5V</text>
 <text x="11.049" y="0.381" size="0.8128" layer="21" font="vector" ratio="17" rot="R90">MACMOD</text>
-<text x="8.128" y="4.064" size="0.6096" layer="51">1</text>
+<text x="7.874" y="4.064" size="0.6096" layer="51">1</text>
+<circle x="8.0264" y="4.318" radius="0.1524" width="0.3048" layer="21"/>
 </plain>
 <attributes>
