File: MACMOD.sch (EAGLE design)
At the start: 5 parts, among them IC1 MCP24AA025E48

Commit message: Improved labels for v1.0 release
Other:
- note added: "(c) Copyright 2017 Freetronics Pty Ltd"
- note added: "V1.0 (1-Aug-2017)"
- note removed: "(c) Copyright 2013 Freetronics Pty Ltd"
- note removed: "V1.0 (4-Jul-2013)"
Changed lines of the file:
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@@
 <plain>
 <text x="144.78" y="12.7" size="3.048" layer="94">Freetronics MAC Address Module</text>
-<text x="215.9" y="6.858" size="1.778" layer="94">V1.0 (4-Jul-2013)</text>
+<text x="215.9" y="6.858" size="1.778" layer="94">V1.0 (1-Aug-2017)</text>
 <text x="144.526" y="6.858" size="1.778" layer="94">www.freetronics.com.au/macmod</text>
 <text x="193.04" y="6.858" size="1.778" layer="94">SKU: MACMOD</text>
@@
 <text x="12.7" y="10.16" size="1.778" layer="94">Open Hardware License</text>
 <text x="12.7" y="7.62" size="1.778" layer="94">www.tapr.org/OHL</text>
-<text x="12.7" y="15.24" size="1.778" layer="94">(c) Copyright 2013 Freetronics Pty Ltd</text>
+<text x="12.7" y="15.24" size="1.778" layer="94">(c) Copyright 2017 Freetronics Pty Ltd</text>
 <text x="137.16" y="111.76" size="1.778" layer="94">VCC</text>
 <text x="137.16" y="109.22" size="1.778" layer="94">SCL</text>
